Commit message: Updated models

File: example_py/MPS_code/models/aliengo_models/urdf/aliengo.urdf (robot description, URDF)
Before this commit: robot aliengo_description, 19 links, 18 joints
Joints:
- joint FL_calf_joint: limit lower=-2.77507351067 upper=-0.645771823238 effort=33.5 velocity=21.0 -> lower=-2.77507351067 upper=-0.645771823238 effort=40 velocity=26.5
- joint FL_hip_joint: limit lower=-1.2217304764 upper=1.2217304764 effort=33.5 velocity=21.0 -> lower=-1.2217304764 upper=1.2217304764 effort=40 velocity=26.5
- joint FL_thigh_joint: limit lower=-1.5707963267948966 upper=1.5707963267948966 effort=33.5 velocity=21.0 -> lower=-1.5707963267948966 upper=1.5707963267948966 effort=40 velocity=26.5
- joint FR_calf_joint: limit lower=-2.77507351067 upper=-0.645771823238 effort=33.5 velocity=21.0 -> lower=-2.77507351067 upper=-0.645771823238 effort=40 velocity=26.5
- joint FR_hip_joint: limit lower=-1.2217304764 upper=1.2217304764 effort=33.5 velocity=21.0 -> lower=-1.2217304764 upper=1.2217304764 effort=40 velocity=26.5
- joint FR_thigh_joint: limit lower=-1.5707963267948966 upper=1.5707963267948966 effort=33.5 velocity=21.0 -> lower=-1.5707963267948966 upper=1.5707963267948966 effort=40 velocity=26.5
- joint RL_calf_joint: limit lower=-2.77507351067 upper=-0.645771823238 effort=33.5 velocity=21.0 -> lower=-2.77507351067 upper=-0.645771823238 effort=40 velocity=26.5
- joint RL_hip_joint: limit lower=-1.2217304764 upper=1.2217304764 effort=33.5 velocity=21.0 -> lower=-1.2217304764 upper=1.2217304764 effort=40 velocity=26.5
- joint RL_thigh_joint: limit lower=-1.5707963267948966 upper=1.5707963267948966 effort=33.5 velocity=21.0 -> lower=-1.5707963267948966 upper=1.5707963267948966 effort=40 velocity=26.5
- joint RR_calf_joint: limit lower=-2.77507351067 upper=-0.645771823238 effort=33.5 velocity=21.0 -> lower=-2.77507351067 upper=-0.645771823238 effort=40 velocity=26.5
- joint RR_hip_joint: limit lower=-1.2217304764 upper=1.2217304764 effort=33.5 velocity=21.0 -> lower=-1.2217304764 upper=1.2217304764 effort=40 velocity=26.5
- joint RR_thigh_joint: limit lower=-1.5707963267948966 upper=1.5707963267948966 effort=33.5 velocity=21.0 -> lower=-1.5707963267948966 upper=1.5707963267948966 effort=40 velocity=26.5
